File: KiCAD/moonboard.kicad_sch (KiCad schematic)
At the start: 0 parts

Commit message: Finished Schematic!
Parts:
- added D1, D2, D3, D4, D5, D6: D_Small, symbol Device:D_Small
- added J1: Conn_01x04_Pin, symbol Connector:Conn_01x04_Pin
- added J2: Conn_01x08_Pin, symbol Connector:Conn_01x08_Pin
- added R1: 10k, symbol Device:R_Small
- added RV1: R_Potentiometer, symbol Device:R_Potentiometer
- added SW1, SW2, SW3, SW4, SW5, SW6: SW_Push_45deg, symbol Switch:SW_Push_45deg
- added U1: XIAO-ESP32-C3-SMD, Seeed_Studio_XIAO_Series:XIAO-ESP32-C3-SMD, symbol PCM_Seeed_Studio_XIAO_Series:XIAO-ESP32-C3-SMD
- added U2: DHT11, Sensor:Aosong_DHT11_5.5x12.0_P2.54mm, symbol Sensor:DHT11
Connections:
- new net: D6.2 (A), SW6.2
- new net: D5.2 (A), SW5.2
- new net: D3.2 (A), SW3.2
- new net: D2.2 (A), SW2.2
- new net: D4.2 (A), SW4.2
- new net: D1.2 (A), SW1.2
- new net +3V3: J1.3 (Pin_3), J2.1 (Pin_1), R1.1, RV1.1, U1.12 (3V3_OUT), U2.1 (VDD)
- new net +5V: U1.14 (VBUS)
- new net COL0: SW1.1, SW4.1, U1.2 (D1)
- new net COL1: SW2.1, SW5.1, U1.3 (D2)
- new net COL2: SW3.1, SW6.1, U1.4 (D3)
- new net DHT11_DATA: R1.2, U1.1 (D0), U2.2 (DATA)
- new net GND: J1.4 (Pin_4), J2.2 (Pin_2), RV1.3, U1.13 (GND), U1.18 (GND), U2.4 (GND)
- new net POT_IN: RV1.2, U1.11 (D10)
- new net ROW0: D1.1 (K), D2.1 (K), D3.1 (K), U1.7 (D6)
- new net ROW1: D4.1 (K), D5.1 (K), D6.1 (K), U1.8 (D7)
- new net SCL: J1.2 (Pin_2), J2.3 (Pin_3), U1.6 (D5)
- new net SDA: J1.1 (Pin_1), J2.4 (Pin_4), U1.5 (D4)
- no-connect marks 0 -> 13
Other:
- note added: "BUTTONS"
- note added: "ESP32-C3"
- note added: "MPU6050"
- note added: "OLED"
- note added: "Potentiometer"
- note added: "TEMP SENSOR"

Commit message: Finished PCB
Parts:
- D1, D2, D3, D4, D5, D6: footprint (none) -> Diode_SMD:D_SOD-123
- J1: footprint (none) -> FootprintsnModels:OLED_SSD1306_I2C_0.96
- J2: footprint (none) -> FootprintsnModels:MODULE_GY-521
- R1: footprint (none) -> Resistor_SMD:R_0805_2012Metric
- RV1: footprint (none) -> FootprintsnModels:RotaryEncoder_Alps_EC11E-Switch_Vertical_H20mm
- SW1, SW2, SW3, SW4, SW5, SW6: footprint (none) -> PCM_ScottoKeebs_Hotswap:Hotswap_MX_1.00u
- U1: footprint Seeed_Studio_XIAO_Series:XIAO-ESP32-C3-SMD -> XIAO_footprints:XIAO-ESP32-C3-SMD
Changed lines of the file:
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@@
 			)
 		)
-		(property "Footprint" ""
+		(property "Footprint" "PCM_ScottoKeebs_Hotswap:Hotswap_MX_1.00u"
 			(at 137.16 55.88 0)
 			(hide yes)
@@
 			)
 		)
-		(property "Footprint" ""
+		(property "Footprint" "Diode_SMD:D_SOD-123"
 			(at 123.19 60.96 90)
 			(hide yes)
@@
 			)
 		)
-		(property "Footprint" ""
+		(property "Footprint" "Diode_SMD:D_SOD-123"
 			(at 139.7 60.96 90)
 			(hide yes)
@@
 			)
 		)
-		(property "Footprint" ""
+		(property "Footprint" "Diode_SMD:D_SOD-123"
 			(at 139.7 40.64 90)
 			(hide yes)
@@
 			)
 		)
-		(property "Footprint" ""
+		(property "Footprint" "FootprintsnModels:RotaryEncoder_Alps_EC11E-Switch_Vertical_H20mm"
 			(at 111.76 113.03 0)
 			(hide yes)
@@
 			)
 		)
-		(property "Footprint" ""
+		(property "Footprint" "Diode_SMD:D_SOD-123"
 			(at 123.19 40.64 90)
 			(hide yes)
@@
 			)
 		)
-		(property "Footprint" ""
+		(property "Footprint" "PCM_ScottoKeebs_Hotswap:Hotswap_MX_1.00u"
 			(at 104.14 55.88 0)
 			(hide yes)
@@
 			)
 		)
-		(property "Footprint" ""
+		(property "Footprint" "PCM_ScottoKeebs_Hotswap:Hotswap_MX_1.00u"
 			(at 120.65 35.56 0)
 			(hide yes)
@@
 			)
 		)
-		(property "Footprint" ""
+		(property "Footprint" "PCM_ScottoKeebs_Hotswap:Hotswap_MX_1.00u"
 			(at 120.65 55.88 0)
 			(hide yes)
@@
 			)
 		)
-		(property "Footprint" ""
+		(property "Footprint" "FootprintsnModels:MODULE_GY-521"
 			(at 101.6 86.36 0)
 			(hide yes)
@@
 			)
 		)
-		(property "Footprint" ""
+		(property "Footprint" "Resistor_SMD:R_0805_2012Metric"
 			(at 53.34 114.3 0)
 			(hide yes)
@@
 			)
 		)
-		(property "Footprint" ""
+		(property "Footprint" "FootprintsnModels:OLED_SSD1306_I2C_0.96"
 			(at 74.93 93.98 0)
 			(hide yes)
@@
 			)
 		)
-		(property "Footprint" ""
+		(property "Footprint" "PCM_ScottoKeebs_Hotswap:Hotswap_MX_1.00u"
 			(at 137.16 35.56 0)
 			(hide yes)
@@
 			)
 		)
-		(property "Footprint" ""
+		(property "Footprint" "Diode_SMD:D_SOD-123"
 			(at 106.68 40.64 90)
 			(hide yes)
@@
 			)
 		)
-		(property "Footprint" ""
+		(property "Footprint" "Diode_SMD:D_SOD-123"
 			(at 106.68 60.96 90)
 			(hide yes)
@@
 			)
 		)
-		(property "Footprint" "Seeed_Studio_XIAO_Series:XIAO-ESP32-C3-SMD"
+		(property "Footprint" "XIAO_footprints:XIAO-ESP32-C3-SMD"
 			(at 16.002 76.454 0)
 			(hide yes)
@@
 			)
 		)
-		(property "Footprint" ""
+		(property "Footprint" "PCM_ScottoKeebs_Hotswap:Hotswap_MX_1.00u"
 			(at 104.14 35.56 0)
 			(hide yes)
