File: KiCAD/_autosave-moonboard.kicad_pcb (KiCad board)
At the start: 2 copper layers, 99.5 x 70.5 mm, 18 parts, among them J1 Conn_01x04_Pin, J2 Conn_01x08_Pin, SW1 SW_Push_45deg, SW2 SW_Push_45deg, SW3 SW_Push_45deg, SW4 SW_Push_45deg, SW5 SW_Push_45deg, SW6 SW_Push_45deg, U1 XIAO-ESP32-C3-SMD, U2 DHT11

Commit message: fixed up PCB, also added 3d models and renders
Parts:
- moved U2 17.9 mm to (205.5, 77.1), turned to 180 degrees
Routing:
- net +3V3: track 167.8 -> 152.4 mm
- net /DHT11_DATA: track 34.9 -> 47.2 mm
